Commit message: [feat] added controllers for all joints and rqt

File: src/mrm_description/urdf/links_joints.xacro (robot description, xacro)
@@ -1,12 +1,22 @@
 <?xml version="1.0"?>
 <robot xmlns:xacro="http://www.ros.org/wiki/xacro">
-    <xacro:macro name="m_joint" params="name type axis_xyz origin_rpy origin_xyz parent child">
+    <xacro:macro name="m_joint" params="name type axis_xyz origin_rpy origin_xyz parent child limit_e limit_l limit_u limit_v">
         <joint name="${name}" type="${type}">
             <axis xyz="${axis_xyz}" />
-            <limit effort="1000.0" lower="-3.14" upper="3.14" velocity="0.5" />
+            <limit effort="${limit_e}" lower="${limit_l}" upper="${limit_u}" velocity="${limit_v}" />
             <origin rpy="${origin_rpy}" xyz="${origin_xyz}" />
             <parent link="${parent}" />
             <child link="${child}" />
         </joint>
+        <transmission name="trans_${name}">
+            <type>transmission_interface/SimpleTransmission</type>
+            <joint name="${name}">
+                <hardwareInterface>hardware_interface/EffortJointInterface</hardwareInterface>
+            </joint>
+            <actuator name="motor_${name}">
+                <hardwareInterface>hardware_interface/EffortJointInterface</hardwareInterface>
+                <mechanicalReduction>1</mechanicalReduction>
+            </actuator>
+        </transmission>
     </xacro:macro>
     <xacro:macro name="m_link_cylinder" params="name origin_xyz origin_rpy radius length mass ixx ixy ixz iyy iyz izz">

File: src/mrm_description/urdf/mrm.xacro (robot description, xacro)
@@ -1,156 +1,163 @@
 <?xml version="1.0"?>
-<robot
-        name="mrm"
+<robot name="mrm"
         xmlns:xacro="http://www.ros.org/wiki/xacro">
-    <!-- BGN - Include -->
-    <xacro:include filename="$(find mrm_description)/urdf/links_joints.xacro" />
-    <xacro:include filename="$(find mrm_description)/urdf/robot_parameters.xacro" />
-    <!-- END - Include -->
-    <!-- BGN - Robot description -->
-    <m_link_box
-            name="${link_00_name}"
-            origin_rpy="0 0 0"
-            origin_xyz="0 0 0"
-            mass="1024"
-            ixx="170.667"
-            ixy="0"
-            ixz="0"
-            iyy="170.667"
-            iyz="0"
-            izz="170.667"
-            size="1 1 1" />
-    <m_joint
-            name="${link_00_name}__${link_01_name}"
-            type="revolute"
-            axis_xyz="0 0 1"
-            origin_rpy="0 0 0"
-            origin_xyz="0 0 0.5"
-            parent="${link_00_name}"
-            child="${link_01_name}" />
-<!-- Transmission for controller -->
-  <transmission name="trans_${link_00_name}__${link_01_name}">
-    <type>transmission_interface/SimpleTransmission</type>
-    <joint name="${link_00_name}__${link_01_name}">
-        <hardwareInterface>hardware_interface/EffortJointInterface</hardwareInterface>
-    </joint>
-    <actuator name="motor_${link_00_name}__${link_01_name}">
-        <hardwareInterface>hardware_interface/EffortJointInterface</hardwareInterface>
-        <mechanicalReduction>1</mechanicalReduction>
-    </actuator>
-  </transmission>
-    <m_link_cylinder
-            name="${link_01_name}"
-            origin_rpy="0 0 0"
-            origin_xyz="0 0 0.2"
-            mass="157.633"
-            ixx="13.235"
-            ixy="0"
-            ixz="0"
-            iyy="13.235"
-            iyz="0"
-            izz="9.655"
-            length="0.4"
-            radius="0.35" />
-    <m_joint
-            name="${link_01_name}__${link_02_name}"
-            type="revolute"
-            axis_xyz="0 1 0"
-            origin_rpy="0 0 0"
-            origin_xyz="0 0 0.4"
-            parent="${link_01_name}"
-            child="${link_02_name}" />
-<!-- Transmission for controller -->
-  <transmission name="trans_${link_01_name}__${link_02_name}">
-    <type>transmission_interface/SimpleTransmission</type>
-    <joint name="${link_01_name}__${link_02_name}">
-        <hardwareInterface>hardware_interface/EffortJointInterface</hardwareInterface>
-    </joint>
-    <actuator name="motor_${link_01_name}__${link_02_name}">
-        <hardwareInterface>hardware_interface/EffortJointInterface</hardwareInterface>
-        <mechanicalReduction>1</mechanicalReduction>
-    </actuator>
-  </transmission>
-    <m_link_cylinder
-            name="${link_02_name}"
-            origin_rpy="0 0 0"
-            origin_xyz="0 0 0.4"
-            mass="57.906"
-            ixx="12.679"
-            ixy="0"
-            ixz="0"
-            iyy="12.679"
-            iyz="0"
-            izz="0.651"
-            radius="0.15"
-            length="0.8" />
-            <!--
-    <m_joint
-            name="${link_02_name}__${link_03_name}"
-            type="revolute"
-            axis_xyz="0 1 0"
-            origin_rpy="0 0 0"
-            origin_xyz="0 0 0.8"
-            parent="${link_02_name}"
-            child="${link_03_name}" />
-    <m_link_cylinder
-            name="${link_03_name}"
-            origin_rpy="0 0 0"
-            origin_xyz="0 0 0.4"
-            mass="57.906"
-            ixx="12.679"
-            ixy="0"
-            ixz="0"
-            iyy="12.679"
-            iyz="0"
-            izz="0.651"
-            radius="0.15"
-            length="0.8" />
-    <m_joint
-            name="${link_03_name}__${link_04_name}"
-            type="revolute"
-            axis_xyz="0 1 0"
-            origin_rpy="0 0 0"
-            origin_xyz="0 0 0.8"
-            parent="${link_03_name}"
-            child="${link_04_name}" />
-    <m_link_cylinder
-            name="${link_04_name}"
-            origin_rpy="0 0 0"
-            origin_xyz="0 0 0.4"
-            mass="57.906"
-            ixx="12.679"
-            ixy="0"
-            ixz="0"
-            iyy="12.679"
-            iyz="0"
-            izz="0.651"
-            radius="0.15"
-            length="0.8" />
-    <m_joint
-            name="${link_04_name}__${link_05_name}"
-            type="revolute"
-            axis_xyz="0 0 1"
-            origin_rpy="0 0 0"
-            origin_xyz="0 0 0.8"
-            parent="${link_04_name}"
-            child="${link_05_name}" />
-    <m_link_cylinder
-            name="${link_05_name}"
-            origin_rpy="0 0 0"
-            origin_xyz="0 0 0.125"
-            mass="18.056"
-            ixx="0.479"
-            ixy="0"
-            ixz="0"
-            iyy="0.479"
-            iyz="0"
-            izz="0.204"
-            radius="0.15"
-            length="0.25" />
-    -->
-<gazebo>
-    <plugin name="gazebo_ros_control" filename="libgazebo_ros_control.so">
-    </plugin>
-</gazebo>
-    <!-- END - Robot description -->
+        <!-- BGN - Include -->
+        <xacro:include filename="$(find mrm_description)/urdf/links_joints.xacro" />
+        <xacro:include filename="$(find mrm_description)/urdf/robot_parameters.xacro" />
+        <!-- END - Include -->
+        <!-- BGN - Robot description -->
+        <m_link_box name="${link_00_name}"
+                origin_rpy="0 0 0"
+                origin_xyz="0 0 0"
+                mass="1024"
+                ixx="170.667"
+                ixy="0"
+                ixz="0"
+                iyy="170.667"
+                iyz="0"
+                izz="170.667"
+                size="1 1 1" />
+        <m_joint name="${link_00_name}__${link_01_name}"
+                type="revolute"
+                axis_xyz="0 0 1"
+                origin_rpy="0 0 0"
+                origin_xyz="0 0 0.5"
+                parent="${link_00_name}"
+                child="${link_01_name}"
+                limit_e="1000"
+                limit_l="-3.14"
+                limit_u="3.14"
+                limit_v="0.5" />
+        <!-- Transmission for controller -->
+        <transmission name="trans_${link_00_name}__${link_01_name}">
+                <type>transmission_interface/SimpleTransmission</type>
+                <joint name="${link_00_name}__${link_01_name}">
+                        <hardwareInterface>hardware_interface/EffortJointInterface</hardwareInterface>
+                </joint>
+                <actuator name="motor_${link_00_name}__${link_01_name}">
+                        <hardwareInterface>hardware_interface/EffortJointInterface</hardwareInterface>
+                        <mechanicalReduction>1</mechanicalReduction>
+                </actuator>
+        </transmission>
+        <m_link_cylinder name="${link_01_name}"
+                origin_rpy="0 0 0"
+                origin_xyz="0 0 0.2"
+                mass="157.633"
+                ixx="13.235"
+                ixy="0"
+                ixz="0"
+                iyy="13.235"
+                iyz="0"
+                izz="9.655"
+                length="0.4"
+                radius="0.35" />
+        <m_joint name="${link_01_name}__${link_02_name}"
+                type="revolute"
+                axis_xyz="0 1 0"
+                origin_rpy="0 0 0"
+                origin_xyz="0 0 0.4"
+                parent="link_01"
+                child="link_02"
+                limit_e="1000"
+                limit_l="0"
+                limit_u="0.5"
+                limit_v="0.5" />
+        <!-- Transmission for controller -->
+        <transmission name="trans_${link_01_name}__${link_02_name}">
+                <type>transmission_interface/SimpleTransmission</type>
+                <joint name="${link_01_name}__${link_02_name}">
+                        <hardwareInterface>hardware_interface/EffortJointInterface</hardwareInterface>
+                </joint>
+                <actuator name="motor_${link_01_name}__${link_02_name}">
+                        <hardwareInterface>hardware_interface/EffortJointInterface</hardwareInterface>
+                        <mechanicalReduction>1</mechanicalReduction>
+                </actuator>
+        </transmission>
+        <m_link_cylinder name="${link_02_name}"
+                origin_rpy="0 0 0"
+                origin_xyz="0 0 0.4"
+                mass="57.906"
+                ixx="12.679"
+                ixy="0"
+                ixz="0"
+                iyy="12.679"
+                iyz="0"
+                izz="0.651"
+                radius="0.15"
+                length="0.8" />
+        <m_joint name="${link_02_name}__${link_03_name}"
+                type="revolute"
+                axis_xyz="0 1 0"
+                origin_rpy="0 0 0"
+                origin_xyz="0 0 0.8"
+                parent="link_02"
+                child="link_03"
+                limit_e="1000"
+                limit_l="0"
+                limit_u="0.75"
+                limit_v="0.5" />
+        <m_link_cylinder name="${link_03_name}"
+                origin_rpy="0 0 0"
+                origin_xyz="0 0 0.4"
+                mass="57.906"
+                ixx="12.679"
+                ixy="0"
+                ixz="0"
+                iyy="12.679"
+                iyz="0"
+                izz="0.651"
+                radius="0.15"
+                length="0.8" />
+        <m_joint name="${link_03_name}__${link_04_name}"
+                type="revolute"
+                axis_xyz="0 1 0"
+                origin_rpy="0 0 0"
+                origin_xyz="0 0 0.8"
+                parent="link_03"
+                child="link_04"
+                limit_e="1000"
+                limit_l="0"
+                limit_u="0.75"
+                limit_v="0.5" />
+        <m_link_cylinder name="${link_04_name}"
+                origin_rpy="0 0 0"
+                origin_xyz="0 0 0.4"
+                mass="57.906"
+                ixx="12.679"
+                ixy="0"
+                ixz="0"
+                iyy="12.679"
+                iyz="0"
+                izz="0.651"
+                radius="0.15"
+                length="0.8" />
+        <m_joint name="${link_04_name}__${link_05_name}"
+                type="revolute"
+                axis_xyz="0 0 1"
+                origin_rpy="0 0 0"
+                origin_xyz="0 0 0.8"
+                parent="link_04"
+                child="link_05"
+                limit_e="1000"
+                limit_l="-3.14"
+                limit_u="3.14"
+                limit_v="0.5" />
+        <m_link_cylinder name="${link_05_name}"
+                origin_rpy="0 0 0"
+                origin_xyz="0 0 0.125"
+                mass="18.056"
+                ixx="0.479"
+                ixy="0"
+                ixz="0"
+                iyy="0.479"
+                iyz="0"
+                izz="0.204"
+                radius="0.15"
+                length="0.25" />
+        <gazebo>
+                <plugin name="gazebo_ros_control"
+                        filename="libgazebo_ros_control.so">
+                </plugin>
+        </gazebo>
+        <!-- END - Robot description -->
 </robot>

Commit message: [final] finished part 1

File: src/mrm_description/urdf/links_joints.xacro (robot description, xacro)
@@ -1,9 +1,15 @@
 <?xml version="1.0"?>
 <robot xmlns:xacro="http://www.ros.org/wiki/xacro">
-    <xacro:macro name="m_joint" params="name type axis_xyz origin_rpy origin_xyz parent child limit_e limit_l limit_u limit_v">
-        <joint name="${name}" type="${type}">
+    <xacro:macro name="m_joint"
+        params="name type axis_xyz origin_rpy origin_xyz parent child limit_e limit_l limit_u limit_v">
+        <joint name="${name}"
+            type="${type}">
             <axis xyz="${axis_xyz}" />
-            <limit effort="${limit_e}" lower="${limit_l}" upper="${limit_u}" velocity="${limit_v}" />
-            <origin rpy="${origin_rpy}" xyz="${origin_xyz}" />
+            <limit effort="${limit_e}"
+                lower="${limit_l}"
+                upper="${limit_u}"
+                velocity="${limit_v}" />
+            <origin rpy="${origin_rpy}"
+                xyz="${origin_xyz}" />
             <parent link="${parent}" />
             <child link="${child}" />
@@ -20,34 +26,53 @@
         </transmission>
     </xacro:macro>
-    <xacro:macro name="m_link_cylinder" params="name origin_xyz origin_rpy radius length mass ixx ixy ixz iyy iyz izz">
+    <xacro:macro name="m_link_cylinder"
+        params="name origin_xyz origin_rpy radius length mass ixx ixy ixz iyy iyz izz">
         <link name="${name}">
             <inertial>
                 <mass value="${mass}" />
-                <origin rpy="${origin_rpy}" xyz="${origin_xyz}" />
-                <inertia ixx="${ixx}" ixy="${ixy}" ixz="${ixz}" iyy="${iyy}" iyz="${iyz}" izz="${izz}" />
+                <origin rpy="${origin_rpy}"
+                    xyz="${origin_xyz}" />
+                <inertia ixx="${ixx}"
+                    ixy="${ixy}"
+                    ixz="${ixz}"
+                    iyy="${iyy}"
+                    iyz="${iyz}"
+                    izz="${izz}" />
             </inertial>
             <collision>
-                <origin rpy="${origin_rpy}" xyz="${origin_xyz}" />
+                <origin rpy="${origin_rpy}"
+                    xyz="${origin_xyz}" />
                 <geometry>
-                    <cylinder radius="${radius}" length="${length}" />
+                    <cylinder radius="${radius}"
+                        length="${length}" />
                 </geometry>
             </collision>
             <visual>
-                <origin rpy="${origin_rpy}" xyz="${origin_xyz}" />
+                <origin rpy="${origin_rpy}"
+                    xyz="${origin_xyz}" />
                 <geometry>
-                    <cylinder radius="${radius}" length="${length}" />
+                    <cylinder radius="${radius}"
+                        length="${length}" />
                 </geometry>
             </visual>
         </link>
     </xacro:macro>
-    <xacro:macro name="m_link_box" params="name origin_xyz origin_rpy size mass ixx ixy ixz iyy iyz izz">
+    <xacro:macro name="m_link_box"
+        params="name origin_xyz origin_rpy size mass ixx ixy ixz iyy iyz izz">
         <link name="${name}">
             <inertial>
                 <mass value="${mass}" />
-                <origin rpy="${origin_rpy}" xyz="${origin_xyz}" />
-                <inertia ixx="${ixx}" ixy="${ixy}" ixz="${ixz}" iyy="${iyy}" iyz="${iyz}" izz="${izz}" />
+                <origin rpy="${origin_rpy}"
+                    xyz="${origin_xyz}" />
+                <inertia ixx="${ixx}"
+                    ixy="${ixy}"
+                    ixz="${ixz}"
+                    iyy="${iyy}"
+                    iyz="${iyz}"
+                    izz="${izz}" />
             </inertial>
             <collision>
-                <origin rpy="${origin_rpy}" xyz="${origin_xyz}" />
+                <origin rpy="${origin_rpy}"
+                    xyz="${origin_xyz}" />
                 <geometry>
                     <box size="${size}" />
@@ -55,5 +80,6 @@
             </collision>
             <visual>
-                <origin rpy="${origin_rpy}" xyz="${origin_xyz}" />
+                <origin rpy="${origin_rpy}"
+                    xyz="${origin_xyz}" />
                 <geometry>
                     <box size="${size}" />
@@ -62,3 +88,36 @@
         </link>
     </xacro:macro>
+    <xacro:macro name="m_link_mesh"
+        params="name origin_xyz origin_rpy meshfile meshscale mass ixx ixy ixz iyy iyz izz">
+        <link name="${name}">
+            <inertial>
+                <mass value="${mass}" />
+                <origin rpy="${origin_rpy}"
+                    xyz="${origin_xyz}" />
+                <inertia ixx="${ixx}"
+                    ixy="${ixy}"
+                    ixz="${ixz}"
+                    iyy="${iyy}"
+                    iyz="${iyz}"
+                    izz="${izz}" />
+            </inertial>
+            <collision>
+                <origin rpy="${origin_rpy}"
+                    xyz="${origin_xyz}" />
+                <geometry>
+                    <mesh filename="${meshfile}"
+                        scale="${meshscale}"/>
+                </geometry>
+            </collision>
+            <visual>
+                <origin rpy="${origin_rpy}"
+                    xyz="${origin_xyz}" />
+                <geometry>
+                    <mesh filename="${meshfile}"
+                        scale="${meshscale}"/>
+                </geometry>
+                <material name="light_black"/>
+            </visual>
+        </link>
+    </xacro:macro>
 </robot>

File: src/mrm_description/urdf/mrm.xacro (robot description, xacro)
@@ -29,18 +29,7 @@
                 limit_u="3.14"
                 limit_v="0.5" />
-        <!-- Transmission for controller -->
-        <transmission name="trans_${link_00_name}__${link_01_name}">
-                <type>transmission_interface/SimpleTransmission</type>
-                <joint name="${link_00_name}__${link_01_name}">
-                        <hardwareInterface>hardware_interface/EffortJointInterface</hardwareInterface>
-                </joint>
-                <actuator name="motor_${link_00_name}__${link_01_name}">
-                        <hardwareInterface>hardware_interface/EffortJointInterface</hardwareInterface>
-                        <mechanicalReduction>1</mechanicalReduction>
-                </actuator>
-        </transmission>
-        <m_link_cylinder name="${link_01_name}"
+        <m_link_mesh name="${link_01_name}"
                 origin_rpy="0 0 0"
-                origin_xyz="0 0 0.2"
+                origin_xyz="0 0 -0.1"
                 mass="157.633"
                 ixx="13.235"
@@ -50,6 +39,6 @@
                 iyz="0"
                 izz="9.655"
-                length="0.4"
-                radius="0.35" />
+                meshfile="package://mrm_description/meshes/Link1-v2.stl"
+                meshscale="0.001 0.001 0.001" />
         <m_joint name="${link_01_name}__${link_02_name}"
                 type="revolute"
@@ -63,15 +52,4 @@
                 limit_u="0.5"
                 limit_v="0.5" />
-        <!-- Transmission for controller -->
-        <transmission name="trans_${link_01_name}__${link_02_name}">
-                <type>transmission_interface/SimpleTransmission</type>
-                <joint name="${link_01_name}__${link_02_name}">
-                        <hardwareInterface>hardware_interface/EffortJointInterface</hardwareInterface>
-                </joint>
-                <actuator name="motor_${link_01_name}__${link_02_name}">
-                        <hardwareInterface>hardware_interface/EffortJointInterface</hardwareInterface>
-                        <mechanicalReduction>1</mechanicalReduction>
-                </actuator>
-        </transmission>
         <m_link_cylinder name="${link_02_name}"
                 origin_rpy="0 0 0"
@@ -132,7 +110,8 @@
                 radius="0.15"
                 length="0.8" />
+        <!-- <m_joint name="${link_04_name}__${link_05_name}" type="revolute" axis_xyz="0 0 1" origin_rpy="0 0 0" origin_xyz="0 0 0.8" parent="link_04" child="link_05" limit_e="1000" limit_l="-3.14" limit_u="3.14" limit_v="0.5" /> -->
         <m_joint name="${link_04_name}__${link_05_name}"
                 type="revolute"
-                axis_xyz="0 0 1"
+                axis_xyz="0 1 0"
                 origin_rpy="0 0 0"
                 origin_xyz="0 0 0.8"
@@ -140,6 +119,6 @@
                 child="link_05"
                 limit_e="1000"
-                limit_l="-3.14"
-                limit_u="3.14"
+                limit_l="-0.75"
+                limit_u="0"
                 limit_v="0.5" />
         <m_link_cylinder name="${link_05_name}"
